File: OpenAmiga500FastRamExpansion.sch (KiCad schematic (older format))
At the start: 35 parts, among them J1 68000_SOCKET, P1 JTAG_CONNECTOR, P99 OSHW_LOGO, U1 68000D, U2 74LS157, U3 74LS157, U4 ATF1502AS-10JU44, U5 HYB5118160BSJ, U6 HYB5118160BSJ, U7 HYB5118160BSJ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

Commit message: Routing complete Ground stitching and some refinements TBD
Parts:
- P1: footprint Connector_PinHeader_2.54mm:PinHeader_2x05_P2.54mm_Vertical -> Connector_IDC:IDC-Header_2x05_P2.54mm_Vertical
- U4: footprint Package_LCC:PLCC-44_THT-Socket -> OpenAmiga500FastRamExpansion:PLCC-44_THT-Socket
Changed lines of the file:
@@
 F 0 "U4" H 6450 9350 50  0000 L CNN
 F 1 "ATF1502AS-10JU44" H 6220 9260 50  0000 L CNN
-F 2 "Package_LCC:PLCC-44_THT-Socket" H 6510 9320 50  0001 C CNN
+F 2 "OpenAmiga500FastRamExpansion:PLCC-44_THT-Socket" H 6510 9320 50  0001 C CNN
 F 3 "DOCUMENTATION" H 6510 9320 50  0001 C CNN
 	1    6510 9320
@@
 F 0 "P1" H 2670 10713 60  0000 C CNN
 F 1 "JTAG_CONNECTOR" H 2670 10615 50  0000 C CNN
-F 2 "Connector_PinHeader_2.54mm:PinHeader_2x05_P2.54mm_Vertical" H 2670 10270 50  0001 C CNN
+F 2 "Connector_IDC:IDC-Header_2x05_P2.54mm_Vertical" H 2670 10270 50  0001 C CNN
 F 3 "" H 2670 10270 50  0001 C CNN
 	1    2670 10270
