File: OpenAmiga500FastRamExpansion.sch (KiCad schematic (older format))
At the start: 35 parts, among them J1 68000_SOCKET, P1 JTAG_CONNECTOR, P99 OSHW_LOGO, U1 68000D, U2 74LS157, U3 74LS157, U4 ATF1502AS-10JU44, U5 HYB5118160BSJ, U6 HYB5118160BSJ, U7 HYB5118160BSJ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

Commit message: Fix #1 and we're ready for V1
Connections:
- wire segments 499 -> 500
Other:
- moved on the sheet: LD1, R4
Changed lines of the file:
@@
 Title "OpenAmiga500FastRamExpansion"
 Date "2019-05-19"
-Rev "1git"
+Rev "1"
 Comp "SukkoPera"
 Comment1 "Based on work by Kipper2K"
@@
 Wire Wire Line
 	11400 10000 11400 10120
-Wire Wire Line
-	11400 10720 11400 10870
-$Comp
-L Device:LED LD1
-U 1 1 5CBAB2B0
-P 11400 10270
-F 0 "LD1" V 11345 10348 50  0000 L CNN
-F 1 "LED" V 11436 10348 50  0000 L CNN
-F 2 "OpenAmiga500FastRamExpansion:LED_0805_HandSoldering_ModSilkS" H 11400 10270 50  0001 C CNN
-F 3 "~" H 11400 10270 50  0001 C CNN
-	1    11400 10270
-	0    1    1    0
-$EndComp
-$Comp
-L Device:R R4
-U 1 1 5CBCAA9F
-P 11400 10570
-F 0 "R4" H 11410 10710 50  0000 L CNN
-F 1 "10k" V 11400 10500 50  0000 L CNN
-F 2 "Resistor_SMD:R_0805_2012Metric_Pad1.15x1.40mm_HandSolder" V 11330 10570 50  0001 C CNN
-F 3 "~" H 11400 10570 50  0001 C CNN
-	1    11400 10570
-	1    0    0    -1
-$EndComp
 Text Notes 11210 9700 0    50   ~ 0
 POWER LED
@@
 Wire Wire Line
 	3620 7660 3190 7660
+$Comp
+L Device:LED LD1
+U 1 1 5CBAB2B0
+P 11400 10625
+F 0 "LD1" V 11345 10703 50  0000 L CNN
+F 1 "LED" V 11436 10703 50  0000 L CNN
+F 2 "OpenAmiga500FastRamExpansion:LED_0805_HandSoldering_ModSilkS" H 11400 10625 50  0001 C CNN
+F 3 "~" H 11400 10625 50  0001 C CNN
+	1    11400 10625
+	0    -1   -1   0
+$EndComp
+Wire Wire Line
+	11400 10775 11400 10870
+Wire Wire Line
+	11400 10420 11400 10475
+$Comp
+L Device:R R4
+U 1 1 5CBCAA9F
+P 11400 10270
+F 0 "R4" H 11470 10270 50  0000 L CNN
+F 1 "10k" V 11400 10200 50  0000 L CNN
+F 2 "Resistor_SMD:R_0805_2012Metric_Pad1.15x1.40mm_HandSolder" V 11330 10270 50  0001 C CNN
+F 3 "~" H 11400 10270 50  0001 C CNN
+	1    11400 10270
+	1    0    0    -1
+$EndComp
 Wire Bus Line
 	8370 3300 8370 7610
