File: OpenAmiga500FastRamExpansion.kicad_pcb (KiCad board)
At the start: 2 copper layers, 100 x 71.5 mm, 35 parts, among them J1 68000_SOCKET, P1 JTAG_CONNECTOR, P99 OSHW_LOGO, U1 68000D, U2 74LS157, U3 74LS157, U4 ATF1502AS-10JU44, U5 HYB5118160BSJ, U6 HYB5118160BSJ, U7 HYB5118160BSJ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

Commit message: Fix #1 and we're ready for V1
Parts:
- moved LD1 4.69 mm to (189.9, 66.8)
- moved R4 4.69 mm to (189.9, 71.5), turned to 180 degrees
Connections:
- LD1 pad 1: VCC -> GND
- R4 pad 1: Net-(LD1-Pad2) -> VCC
- R4 pad 2: GND -> Net-(LD1-Pad2)
Changed lines of the file:
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@@
     (thickness 1.6)
     (drawings 22)
-    (tracks 1488)
+    (tracks 1486)
     (zones 0)
     (modules 35)
@@
     (title OpenAmiga500FastRamExpansion)
     (date 2019-05-19)
-    (rev 1git)
+    (rev 1)
     (company SukkoPera)
     (comment 1 "Based on work by Kipper2K")
@@
     (0 F.Cu signal)
     (31 B.Cu signal)
-    (34 B.Paste user)
     (36 B.SilkS user)
     (37 F.SilkS user)
@@
     (39 F.Mask user)
     (44 Edge.Cuts user)
-    (45 Margin user hide)
-    (46 B.CrtYd user hide)
-    (47 F.CrtYd user hide)
+    (45 Margin user)
+    (46 B.CrtYd user)
+    (47 F.CrtYd user)
     (49 F.Fab user)
   )
@@
   )
   (module OpenAmiga500FastRamExpansion:LED_0805_HandSoldering_ModSilkS (layer F.Cu)
-    (at 189.865 71.501 180)
+    (at 189.865 66.811 180)
     (descr "Resistor SMD 0805, hand soldering")
     (tags "resistor 0805")
     (attr smd)
-    (fp_text reference LD1 (at 0 -1.914 180) (layer F.SilkS)
+    (fp_text reference LD1 (at 0 1.787 180) (layer F.SilkS)
       (effects (font (size 1 1) (thickness 0.15)))
     )
@@
       (net 67 "Net-(LD1-Pad2)"))
     (pad 1 smd rect (at -1.35 0 180) (size 1.5 1.3) (layers F.Cu F.Mask)
-      (net 19 VCC))
+      (net 18 GND))
     (model ${KISYS3DMOD}/LEDs.3dshapes/LED_0805.wrl
       (at (xyz 0 0 0))
@@
   )
   (module Resistor_SMD:R_0805_2012Metric_Pad1.15x1.40mm_HandSolder (layer F.Cu)
-    (at 189.865 66.811)
+    (at 189.865 71.501 180)
     (descr "Resistor SMD 0805 (2012 Metric), square (rectangular) end terminal, IPC_7351 nominal with elongated pad for handsoldering. (Body size source: https://docs.google.com/spreadsheets/d/1BsfQQcO9C6DZCsRaXUlFlo91Tg2WpOkGARC1WS5S8t0/edit?usp=sharing), generated with kicad-footprint-generator")
     (tags "resistor handsolder")
     (attr smd)
-    (fp_text reference R4 (at 0.054 1.952843) (layer F.SilkS)
+    (fp_text reference R4 (at 0 1.651) (layer F.SilkS)
       (effects (font (size 1 1) (thickness 0.15)))
     )
@@
     (fp_line (start -1 -0.6) (end 1 -0.6) (layer F.Fab) (width 0.1))
     (fp_line (start -1 0.6) (end -1 -0.6) (layer F.Fab) (width 0.1))
-    (pad 2 smd roundrect (at 1.025 0) (size 1.15 1.4) (layers F.Cu F.Paste F.Mask) (roundrect_rratio 0.217391)
-      (net 18 GND))
-    (pad 1 smd roundrect (at -1.025 0) (size 1.15 1.4) (layers F.Cu F.Paste F.Mask) (roundrect_rratio 0.217391)
+    (pad 2 smd roundrect (at 1.025 0 180) (size 1.15 1.4) (layers F.Cu F.Paste F.Mask) (roundrect_rratio 0.217391)
       (net 67 "Net-(LD1-Pad2)"))
+    (pad 1 smd roundrect (at -1.025 0 180) (size 1.15 1.4) (layers F.Cu F.Paste F.Mask) (roundrect_rratio 0.217391)
+      (net 19 VCC))
     (model ${KISYS3DMOD}/Resistor_SMD.3dshapes/R_0805_2012Metric.wrl
       (at (xyz 0 0 0))
@@
   (segment (start 184.023 96.012) (end 183.388 96.012) (width 0.5) (layer F.Cu) (net 19))
   (segment (start 188.916578 96.012) (end 184.023 96.012) (width 0.5) (layer F.Cu) (net 19))
-  (segment (start 195.7705 94.176315) (end 195.7705 94.742) (width 0.5) (layer F.Cu) (net 19))
-  (segment (start 195.7705 72.136) (end 195.7705 94.176315) (width 0.5) (layer F.Cu) (net 19))
-  (segment (start 195.1355 71.501) (end 195.7705 72.136) (width 0.5) (layer F.Cu) (net 19))
   (segment (start 168.402 117.19229) (end 170.055 117.19229) (width 0.5) (layer F.Cu) (net 19) (status 20))
-  (segment (start 193.167 71.501) (end 191.215 71.501) (width 0.5) (layer F.Cu) (net 19) (status 20))
-  (segment (start 192.866 71.501) (end 193.167 71.501) (width 0.5) (layer F.Cu) (net 19))
-  (segment (start 193.167 71.501) (end 195.1355 71.501) (width 0.5) (layer F.Cu) (net 19))
   (segment (start 101.219 117.1956) (end 103.124 117.1956) (width 0.5) (layer B.Cu) (net 19) (status 20))
   (segment (start 140.21 55.634) (end 140.21 54.102) (width 0.5) (layer B.Cu) (net 19) (status 10))
@@
   (segment (start 101.219 53.467) (end 100.457 54.229) (width 0.5) (layer B.Cu) (net 19))
   (segment (start 100.457 116.4336) (end 101.219 117.1956) (width 0.5) (layer B.Cu) (net 19))
+  (segment (start 192.866 71.501) (end 190.89 71.501) (width 0.5) (layer F.Cu) (net 19))
+  (segment (start 195.1355 71.501) (end 192.866 71.501) (width 0.5) (layer F.Cu) (net 19))
+  (segment (start 195.7705 94.742) (end 195.7705 72.136) (width 0.5) (layer F.Cu) (net 19))
+  (segment (start 195.7705 72.136) (end 195.1355 71.501) (width 0.5) (layer F.Cu) (net 19))
   (segment (start 145.29 78.494) (end 145.29 82.05) (width 0.2) (layer F.Cu) (net 20) (status 30))
   (segment (start 180.848 96.52) (end 180.848 104.902) (width 0.2) (layer F.Cu) (net 20) (status 20))
@@
   (segment (start 151.003 109.482) (end 151.750998 109.482) (width 0.2) (layer F.Cu) (net 66))
   (segment (start 148.669856 109.482) (end 151.003 109.482) (width 0.2) (layer F.Cu) (net 66) (status 10))
-  (segment (start 188.84 66.811) (end 188.84 69.0335) (width 0.2) (layer F.Cu) (net 67) (status 10))
-  (segment (start 188.515 69.3585) (end 188.515 71.501) (width 0.2) (layer F.Cu) (net 67) (status 20))
-  (segment (start 188.84 69.0335) (end 188.515 69.3585) (width 0.2) (layer F.Cu) (net 67))
+  (segment (start 188.515 66.811) (end 188.515 68.881) (width 0.2) (layer F.Cu) (net 67))
+  (segment (start 188.84 69.206) (end 188.84 71.501) (width 0.2) (layer F.Cu) (net 67))
+  (segment (start 188.515 68.881) (end 188.84 69.206) (width 0.2) (layer F.Cu) (net 67))
   (segment (start 124.97 79.894) (end 124.97 82.05) (width 0.2) (layer F.Cu) (net 68) (status 20))
   (segment (start 124.97 78.494) (end 124.97 79.894) (width 0.2) (layer F.Cu) (net 68) (status 10))
